File: hardware/P2.kicad_pcb (KiCad board)
At the start: 2 copper layers, 27.9 x 109 mm, 18 parts

Commit message: change pkg
Parts:
- C2: footprint Capacitor_SMD:C_0603_1608Metric -> Capacitor_SMD:C_0805_2012Metric
- C3: footprint Capacitor_SMD:C_0402_1005Metric -> Capacitor_SMD:C_0805_2012Metric
- Regulator1: renamed from Voltage Regulator
- moved C2 1.07 mm to (146.9, 112.3)
- renumbered ESC to ESC1, Radio to Radio1, TX0 to TP1, RX0 to TP2, GND to TP3, Pico to U1
Routing:
- net Net-(Regulator1-BST): track 6.39 -> 5.77 mm
- net GND: track 21.3 -> 20.8 mm
