File: hardware/_autosave-P2.kicad_sch (KiCad schematic)
At the start: 24 parts, among them J1 UART, U1 Pico

Commit message: pcb v1, and production files
Parts:
- removed TP3: GND, TestPoint:TestPoint_Pad_D2.0mm, symbol Connector:TestPoint
- H5, H6: footprint MountingHole:MountingHole_3.2mm_M3 -> MountingHole:MountingHole_3.2mm_M3_Pad_Via
Connections:
- net at ESC1. (MOTOR_D): now also U5. (VCC)
- new net: BT1.2 (-), C1.1, ESC1. (MOTOR_D), U2. (VCC), U4. (VCC), U5. (VCC), U6. (VCC)
- new net: BT1.1 (+), C1.2, ESC1. (MOTOR_D), U2. (VCC), U4. (VCC), U5. (VCC), U6. (VCC)
Changed lines of the file:
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@@
       (effects (font (size 1.27 1.27)) (justify left) hide)
     )
-    (property "Footprint" "MountingHole:MountingHole_3.2mm_M3" (at 124.46 101.6 0)
+    (property "Footprint" "MountingHole:MountingHole_3.2mm_M3_Pad_Via" (at 124.46 101.6 0)
       (effects (font (size 1.27 1.27)) hide)
     )
@@
         (path "/4a9076d5-b6ca-4a4c-83f2-7c8fbd6ec85a"
           (reference "#PWR012") (unit 1)
-        )
-      )
-    )
-  )
-  (symbol (lib_id "power:GND") (at 198.12 48.26 0) (unit 1)
-    (in_bom yes) (on_board yes) (dnp no) (fields_autoplaced)
-    (property "Reference" "#PWR016" (at 198.12 54.61 0)
-      (effects (font (size 1.27 1.27)) hide)
-    )
-    (property "Value" "GND" (at 198.12 53.34 0)
-      (effects (font (size 1.27 1.27)))
-    )
-    (property "Footprint" "" (at 198.12 48.26 0)
-      (effects (font (size 1.27 1.27)) hide)
-    )
-    (property "Datasheet" "" (at 198.12 48.26 0)
-      (effects (font (size 1.27 1.27)) hide)
-    )
-    (pin "1")
-    (instances
-      (project "P2"
-        (path "/4a9076d5-b6ca-4a4c-83f2-7c8fbd6ec85a"
-          (reference "#PWR016") (unit 1)
         )
       )
@@
       (effects (font (size 1.27 1.27)) (justify left) hide)
     )
-    (property "Footprint" "MountingHole:MountingHole_3.2mm_M3" (at 124.46 95.25 0)
+    (property "Footprint" "MountingHole:MountingHole_3.2mm_M3_Pad_Via" (at 124.46 95.25 0)
       (effects (font (size 1.27 1.27)) hide)
     )
@@
         )
       )
-    )
-  )
-  (symbol (lib_id "Connector:TestPoint") (at 198.12 48.26 90) (unit 1)
-    (in_bom yes) (on_board yes) (dnp no) (fields_autoplaced)
-    (property "Reference" "TP3" (at 194.818 43.18 90)
-      (effects (font (size 1.27 1.27)) hide)
-    )
-    (property "Value" "GND" (at 194.818 45.72 90)
-      (effects (font (size 1.27 1.27)))
-    )
-    (property "Footprint" "TestPoint:TestPoint_Pad_D2.0mm" (at 198.12 43.18 0)
-      (effects (font (size 1.27 1.27)) hide)
-    )
-    (property "Datasheet" "~" (at 198.12 43.18 0)
-      (effects (font (size 1.27 1.27)) hide)
-    )
-    (pin "1")
-    (instances
-      (project "P2"
-        (path "/4a9076d5-b6ca-4a4c-83f2-7c8fbd6ec85a"
-          (reference "TP3") (unit 1)
-        )
-      )
